File: DemoBoard_SensorForTemp&Rh_IntegratedWithMCU/CR2477 Module.kicad_sch (KiCad schematic)
At the start: 6 parts, among them J1 Batt_Pos_01x01_Pin, J2 Batt_Neg_01x01_Pin

Commit message: Demo_V0.1
Parts:
- C1, C2, C4, C5: symbol PCM_Capacitor_AKL:C_0603 -> Library:C_0603
- J1, J2: symbol Connector:Conn_01x01_Pin -> Library:Conn_01x01_Pin
Changed lines of the file:
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@@
 	)
 	(symbol
-		(lib_id "PCM_Capacitor_AKL:C_0603")
+		(lib_id "Library:C_0603")
 		(at 99.06 78.74 0)
 		(unit 1)
@@
 	)
 	(symbol
-		(lib_id "PCM_Capacitor_AKL:C_0603")
+		(lib_id "Library:C_0603")
 		(at 83.82 78.74 0)
 		(unit 1)
@@
 	)
 	(symbol
-		(lib_id "PCM_Capacitor_AKL:C_0603")
+		(lib_id "Library:C_0603")
 		(at 114.3 78.74 0)
 		(unit 1)
@@
 	)
 	(symbol
-		(lib_id "Connector:Conn_01x01_Pin")
+		(lib_id "Library:Conn_01x01_Pin")
 		(at 53.34 73.66 0)
 		(unit 1)
@@
 	)
 	(symbol
-		(lib_id "Connector:Conn_01x01_Pin")
+		(lib_id "Library:Conn_01x01_Pin")
 		(at 53.34 83.82 0)
 		(unit 1)
@@
 	)
 	(symbol
-		(lib_id "PCM_Capacitor_AKL:C_0603")
+		(lib_id "Library:C_0603")
 		(at 68.58 78.74 0)
 		(unit 1)
