File: DemoBoard_SensorForTemp&Rh_IntegratedWithMCU/DemoBoard_SensorForTemp&Rh_IntegratedWithMCU.kicad_pcb (KiCad board)
At the start: 2 copper layers, 88.9 x 88.9 mm, 56 parts, among them J1 Batt_Pos_01x01_Pin, J2 Batt_Neg_01x01_Pin, J3 EPD_OPM015BG_1.54, Q1 SI1304BDL

Commit message: Demo_V0.1
Parts:
- added nCS: TestPad_3x2mm_forTestHook, Library:TestPad_3x2mm_forTestHook, B.Cu at (138.5, 110.0)
- added nDC: TestPad_3x2mm_forTestHook, Library:TestPad_3x2mm_forTestHook, B.Cu at (130.7, 104.5)
- C1, C12, C14, C2, C3, C4, C5: footprint PCM_Capacitor_SMD_AKL:C_0603_1608Metric_Pad1.05x0.95mm_HandSolder -> Library:C_0603_1608Metric_Pad1.05x0.95mm_HandSolder
- C10, C11, C13, C15, C16, C17, C18, C19, C20, C21, C6, C7, C8, C9: footprint PCM_Capacitor_SMD_AKL:C_0402_1005Metric_Pad0.74x0.62mm_HandSolder -> Library:C_0402_1005Metric_Pad0.74x0.62mm_HandSolder
- D1, D2, D3: footprint PCM_Diode_SMD_AKL:D_SOD-123F -> Library:D_SOD-123F
- J1: footprint Battery:BatteryContactSpring_PODING_BC-1120-X-X -> Library:BatteryContactSpring_PODING_BC-1120-X-X
- J2: footprint Battery:BatteryContactSpring_PODING_BC-1122-X-X -> Library:BatteryContactSpring_PODING_BC-1122-X-X
- J3: footprint Connector_FFC-FPC:Hirose_FH34SRJ-24S-0.5SH(50)_1x24_P0.50mm_Horizontal -> Library:Hirose_FH34SRJ-24S-0.5SH(50)_1x24_P0.50mm_Horizontal
- JP1: footprint Jumper:SolderJumper-3_P1.3mm_Open_RoundedPad1.0x1.5mm_NumberLabels -> Library:SolderJumper-3_P1.3mm_Open_RoundedPad1.0x1.5mm_NumberLabels
- JP2: footprint Jumper:SolderJumper-2_P1.3mm_Open_TrianglePad1.0x1.5mm -> Library:SolderJumper-2_P1.3mm_Open_TrianglePad1.0x1.5mm
- L1: footprint PCM_Inductor_SMD_Handsoldering_AKL:L_Taiyo-Yuden_NR-40xx_BigPads -> Library:L_Taiyo-Yuden_NR-40xx_BigPads
- Q1: footprint Package_TO_SOT_SMD:SOT-323_SC-70 -> Library:SOT-323_SC-70
- R1, R2, R3, R4, R5, R6, R7: footprint PCM_Resistor_SMD_AKL:R_0402_1005Metric_Pad0.72x0.64mm_HandSolder -> Library:R_0402_1005Metric_Pad0.72x0.64mm_HandSolder
- Template_BATT: renamed from REF**; footprint Battery:BatteryHolder_MYOUNG_BS-24-A1AJ009_CR2477 -> Library:BatteryHolder_MYOUNG_BS-24-A1AJ009_CR2477
- U2: footprint E104-BT01_Bluetooth:PE104-BT01 -> Library:PE104-BT01
- U3: footprint Package_LGA:LGA-6_3x3mm_P1.00mm -> Library:LGA-6_3x3mm_P1.00mm
- U4: footprint PCM_Package_DFN_QFN_AKL:QFN-20-1EP_3x3mm_P0.4mm_EP1.65x1.65mm_ThermalVias -> Library:QFN-20-1EP_3x3mm_P0.4mm_EP1.65x1.65mm_ThermalVias
- turned C19 to 135 degrees
Connections:
- net Net-(J3-Pin_18) renamed /E-Ink Driver/VDDD
- J3 pad 4: unconnected-(J3-Pin_4-Pad4) -> /E-Ink Driver/VDHR
Routing:
- net /E-Ink Driver/RST: track 32.8 -> 34.6 mm
- net /E-Ink Driver/nDC: track 34.1 -> 35.7 mm
- net Net-(D3-A): track 13.2 -> 12.5 mm
- net GND: track 491.2 -> 491.8 mm
- net /E-Ink Driver/nSDA: track 41.0 -> 41.5 mm
