File: DemoBoard_SensorForTemp&Rh_IntegratedWithMCU/E-Ink Driver.kicad_sch (KiCad schematic)
At the start: 20 parts, among them J3 EPD_OPM015BG_1.54, Q1 SI1304BDL

Commit message: Demo_V0.1
Parts:
- removed J3: EPD_OPM015BG_1.54, Connector_FFC-FPC:Hirose_FH34SRJ-24S-0.5SH(50)_1x24_P0.50mm_Horizontal, symbol Connector:Conn_01x24_Pin
- added J3: EPD_OPM015BG_1.54, Connector_FFC-FPC:Hirose_FH34SRJ-24S-0.5SH(50)_1x24_P0.50mm_Horizontal, symbol Library:Conn_01x24_MountingPin
- added NT1: NetTie_4_Cross, symbol Library:NetTie_4_Cross
- C10, C16, C17, C18, C19, C20, C21, C6, C7, C8, C9: symbol Device:C_Small -> Library:C_Small
- D1, D2, D3: symbol PCM_Diode_Schottky_AKL:MBR0530 -> Library:MBR0530
- JP1: symbol Jumper:Jumper_3_Open -> Library:Jumper_3_Open
- L1: symbol Device:L_Small -> Library:L_Small
- Q1: symbol Device:Q_NMOS_GSD -> Library:Q_NMOS_GSD
- R3, R6: symbol Device:R_Small -> Library:R_Small
Connections:
- net BS: now also J3.8 (Pin_8)
- net BUSY: now also J3.9 (Pin_9)
- net GDR: now also J3.2 (Pin_2)
- net PREVGH: now also J3.21 (Pin_21)
- net PREVGL: now also J3.23 (Pin_23)
- net RESE: now also J3.3 (Pin_3)
- net SPI_CS: now also J3.12 (Pin_12)
- net SPI_SCK: now also J3.13 (Pin_13)
- net SPI_SDA: now also J3.14 (Pin_14)
- net TSCL: now also J3.6 (Pin_6)
- net TSDA: now also J3.7 (Pin_7)
- net VCOM: now also J3.24 (Pin_24)
- net VDD: now also J3.15 (Pin_15), J3.16 (Pin_16)
- net VPP: now also J3.19 (Pin_19)
- net VSH: now also J3.20 (Pin_20)
- net VSL: now also J3.22 (Pin_22)
- net VSS: now also J3.17 (Pin_17), J3.MP (MountPin)
- net nDC: now also J3.11 (Pin_11)
- net nRST: now also J3.10 (Pin_10)
- net at C17.2: now also J3.5 (Pin_5)
- net VDDD: now reaches C10.2
- net VDDD: now also J3.18 (Pin_18)
- new net VDHR: J3.4 (Pin_4)
- no-connect marks 4 -> 9
