File: DemoBoard_SensorForTemp&Rh_IntegratedWithMCU/E104-BT01.kicad_sch (KiCad schematic)
At the start: 1 part

Commit message: Demo_V0.1
Parts:
- U2: symbol E104-BT01:E104-BT01 -> Library:E104-BT01
Changed lines of the file:
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@@
 	)
 	(symbol
-		(lib_id "E104-BT01:E104-BT01")
+		(lib_id "Library:E104-BT01")
 		(at 53.34 49.53 0)
 		(unit 1)
