File: DemoBoard_SensorForTemp&Rh_IntegratedWithMCU/HC32L110_QFN20.kicad_sch (KiCad schematic)
At the start: 16 parts

Commit message: Demo_V0.1
Parts:
- C11, C12, C13, C14, C15: symbol Device:C_Small -> Library:C_Small
- JP2: symbol Jumper:Jumper_2_Small_Open -> Library:Jumper_2_Small_Open
- R1, R2, R4, R5: symbol Device:R_Small -> Library:R_Small
- TP10, TP6, TP7, TP8, TP9: symbol Connector:TestPoint_Alt -> Library:TestPoint_Alt
- U4: symbol HC32L110C6UA_QFN20:HC32L110C6UA-QFN20 -> Library:HC32L110C6UA-QFN20
Changed lines of the file:
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@@
 	)
 	(symbol
-		(lib_id "Connector:TestPoint_Alt")
+		(lib_id "Library:TestPoint_Alt")
 		(at 259.08 40.64 90)
 		(unit 1)
@@
 	)
 	(symbol
-		(lib_id "Device:C_Small")
+		(lib_id "Library:C_Small")
 		(at 194.31 36.83 0)
 		(unit 1)
@@
 	)
 	(symbol
-		(lib_id "Connector:TestPoint_Alt")
+		(lib_id "Library:TestPoint_Alt")
 		(at 237.49 48.26 90)
 		(unit 1)
@@
 	)
 	(symbol
-		(lib_id "Device:C_Small")
+		(lib_id "Library:C_Small")
 		(at 177.8 36.83 0)
 		(unit 1)
@@
 	)
 	(symbol
-		(lib_id "Device:C_Small")
+		(lib_id "Library:C_Small")
 		(at 201.93 36.83 0)
 		(unit 1)
@@
 	)
 	(symbol
-		(lib_id "Jumper:Jumper_2_Small_Open")
+		(lib_id "Library:Jumper_2_Small_Open")
 		(at 149.86 43.18 0)
 		(unit 1)
@@
 	)
 	(symbol
-		(lib_id "Device:C_Small")
+		(lib_id "Library:C_Small")
 		(at 149.86 36.83 90)
 		(unit 1)
@@
 	)
 	(symbol
-		(lib_id "Device:C_Small")
+		(lib_id "Library:C_Small")
 		(at 185.42 36.83 0)
 		(unit 1)
@@
 	)
 	(symbol
-		(lib_id "Device:R_Small")
+		(lib_id "Library:R_Small")
 		(at 246.38 72.39 90)
 		(unit 1)
@@
 	)
 	(symbol
-		(lib_id "Connector:TestPoint_Alt")
+		(lib_id "Library:TestPoint_Alt")
 		(at 237.49 40.64 90)
 		(unit 1)
@@
 	)
 	(symbol
-		(lib_id "Connector:TestPoint_Alt")
+		(lib_id "Library:TestPoint_Alt")
 		(at 237.49 33.02 90)
 		(unit 1)
@@
 	)
 	(symbol
-		(lib_id "Device:R_Small")
+		(lib_id "Library:R_Small")
 		(at 140.97 36.83 90)
 		(unit 1)
@@
 	)
 	(symbol
-		(lib_id "HC32L110C6UA_QFN20:HC32L110C6UA-QFN20")
+		(lib_id "Library:HC32L110C6UA-QFN20")
 		(at 143.51 87.63 0)
 		(unit 1)
@@
 	)
 	(symbol
-		(lib_id "Connector:TestPoint_Alt")
+		(lib_id "Library:TestPoint_Alt")
 		(at 259.08 33.02 90)
 		(unit 1)
@@
 	)
 	(symbol
-		(lib_id "Device:R_Small")
+		(lib_id "Library:R_Small")
 		(at 246.38 67.31 90)
 		(unit 1)
@@
 	)
 	(symbol
-		(lib_id "Device:R_Small")
+		(lib_id "Library:R_Small")
 		(at 246.38 95.25 90)
 		(unit 1)
