File: DemoBoard_SensorForTemp&Rh_IntegratedWithMCU/HierSch/Demo_AHT20.kicad_sch (KiCad schematic)
At the start: 3 parts

Commit message: Demo_V0.1
Parts:
- C3: symbol Device:C_Small -> Library:C_Small
- R7: symbol Device:R_Small -> Library:R_Small
- U3: symbol TI HDC3022:AHT20 -> Library:AHT20
Changed lines of the file:
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@@
 	)
 	(symbol
-		(lib_id "TI HDC3022:AHT20")
+		(lib_id "Library:AHT20")
 		(at 71.12 64.77 0)
 		(unit 1)
@@
 	)
 	(symbol
-		(lib_id "Device:R_Small")
+		(lib_id "Library:R_Small")
 		(at 44.45 60.96 90)
 		(unit 1)
@@
 	)
 	(symbol
-		(lib_id "Device:C_Small")
+		(lib_id "Library:C_Small")
 		(at 53.34 64.77 0)
 		(unit 1)
